Commit message: fixed an aruco marker on top of manipulator's end-effector

File: src/tool_tracker/urdf/panda.urdf (robot description, URDF)
Before this commit: robot panda, 12 links, 11 joints
Links:
- added link panda_marker, mass 1; collision box size=0.06 0.06 0.002; visual mesh filename=package://tool_tracker/meshes/Aruco_block.dae scale=1 1 1
Joints:
- added joint panda_hand_marker_joint: type fixed, parent panda_hand, child panda_marker, origin xyz=0.068 0 0.068 rpy=0 3.14159265359 0, axis 1 0 0

Commit message: Placed the marker and camera in appropriate positions

File: src/tool_tracker/urdf/panda.urdf (robot description, URDF)
Before this commit: robot panda, 13 links, 12 joints
Joints:
- joint panda_hand_marker_joint: origin xyz=0.068 0 0.068 rpy=0 3.14159265359 0 -> xyz=0.020 0 0.038 rpy=0 1.57079632679 0

File: src/tool_tracker/urdf/simulation_scene.xacro (robot description, xacro)
@@ -61,5 +61,6 @@
     <parent link="world"/>
     <child link="camera_link"/>
-    <origin xyz="1.15 -1.5 1.3" rpy="0 0.356 2.111"/>
+    <!-- Centered on the robot's forward (+X) axis, aimed down at the work area. -->
+    <origin xyz="1.5 0 1.15" rpy="0 0.3 3.14159265359"/>
   </joint>
   <link name="camera_link_optical"></link>
@@ -67,5 +68,4 @@
     <parent link="camera_link"/>
     <child link="camera_link_optical"/>
-    <!-- Standard ROS to Optical Frame Transform: -90 deg roll, -90 deg yaw -->
     <origin xyz="0 0 0" rpy="-1.57079632679 0 -1.57079632679"/>
   </joint>

Commit message: Impletemented the AprilTag detection algorithm

File: src/tool_tracker/urdf/panda.urdf (robot description, URDF)
Before this commit: robot panda, 13 links, 12 joints
Links:
- link panda_marker: geometry collision box size=0.08 0.08 0.002; visual mesh filename=package://tool_tracker/meshes/Aruco_block.dae scale=1.333333 1.333333 1

File: src/tool_tracker/urdf/simulation_scene.xacro (robot description, xacro)
@@ -61,6 +61,6 @@
     <parent link="world"/>
     <child link="camera_link"/>
-    <!-- Centered on the robot's forward (+X) axis, aimed down at the work area. -->
-    <origin xyz="1.5 0 1.15" rpy="0 0.3 3.14159265359"/>
+    <!-- In front of the robot, aimed down toward the center of the arm workspace. -->
+    <origin xyz="1.2 0 1.2" rpy="0 0.5 3.14159265359"/>
   </joint>
   <link name="camera_link_optical"></link>

Commit message: Changed marker to 26h11; modifed the trajectory to move the joint 3 move left/right and modified cam's position accordingly

File: src/tool_tracker/urdf/panda.urdf (robot description, URDF)
Before this commit: robot panda, 13 links, 12 joints
Joints:
- joint panda_hand_marker_joint: origin xyz=0.020 0 0.038 rpy=0 1.57079632679 0 -> xyz=0.050 0 0.050 rpy=0 1.57079632679 0

File: src/tool_tracker/urdf/simulation_scene.xacro (robot description, xacro)
@@ -61,6 +61,6 @@
     <parent link="world"/>
     <child link="camera_link"/>
-    <!-- In front of the robot, aimed down toward the center of the arm workspace. -->
-    <origin xyz="1.2 0 1.2" rpy="0 0.5 3.14159265359"/>
+    <!-- In front of the raised marker path, centered and aimed slightly down. -->
+    <origin xyz="1.35 -0.12 0.37" rpy="0 0 3.14159265359"/>
   </joint>
   <link name="camera_link_optical"></link>
