Commit message: resolved the issue in launching the robot in gazebo

File: src/tool_tracker/urdf/simulation_scene.xacro (robot description, xacro)
@@ -2,5 +2,5 @@
 <robot name="panda_vision_stage" xmlns:xacro="http://www.ros.org/wiki/xacro">
   <!-- 1. Include Pre-installed Panda Xacro -->
-  <xacro:include filename="$(find moveit_resources_panda_description)/urdf/panda.urdf" />
+  <xacro:include filename="$(find tool_tracker)/urdf/panda.urdf" />
   <!-- 2. Single Root Link Definition -->
   <link name="world"/>
@@ -15,4 +15,14 @@
       <geometry><box size="0.05 0.05 0.05"/></geometry>
     </visual>
+    <collision>
+      <geometry>
+        <box size="0.05 0.05 0.05"/>
+      </geometry>
+    </collision>
+    <inertial>
+      <origin xyz="0 0 0" rpy="0 0 0"/>
+      <mass value="1.0"/>
+      <inertia ixx="0.01" iyy="0.01" izz="0.01" ixy="0" ixz="0" iyz="0"/>
+    </inertial>
   </link>
   <joint name="world_to_camera" type="fixed">
@@ -24,5 +34,7 @@
   <gazebo reference="camera_link">
     <sensor type="camera" name="overhead_camera">
+      <always_on>true</always_on>
       <update_rate>30.0</update_rate>
+      <topic>camera/image_raw</topic>
       <camera>
         <horizontal_fov>1.047</horizontal_fov>
@@ -32,10 +44,9 @@
           <format>R8G8B8</format>
         </image>
+        <clip>
+          <far>0.1</far>
+          <near>100.0</near>
+        </clip>
       </camera>
-      <plugin name="camera_controller" filename="libgazebo_ros_camera.so">
-        <ros>
-          <remapping>~/image_raw:=/camera/image_raw</remapping>
-        </ros>
-      </plugin>
     </sensor>
   </gazebo>

Commit message: positioned the model 0.1 along z axis; commented the control tags in simulation_scene xacro file

File: src/tool_tracker/urdf/simulation_scene.xacro (robot description, xacro)
@@ -3,4 +3,9 @@
   <!-- 1. Include Pre-installed Panda Xacro -->
   <xacro:include filename="$(find tool_tracker)/urdf/panda.urdf" />
+  <!-- <xacro:include filename="$(find moveit_resources_panda_description)/urdf/panda.urdf" />
+  <xacro:include filename="$(find moveit_resources_panda_description)/urdf/panda_ros2_control.xacro" /> -->
+  <!-- <xacro:panda_ros2_control
+    name="PandaGazeboHardware"
+    plugin_name="gz_ros2_control/GazeboSimSystem" /> -->
   <!-- 2. Single Root Link Definition -->
   <link name="world"/>
@@ -29,8 +34,16 @@
     <parent link="world"/>
     <child link="camera_link"/>
-    <origin xyz="0.5 0.0 0.8" rpy="0 0.785 3.14159"/>
+    <origin xyz="0.8 0.0 1.2" rpy="0 0.785 3.14159"/>
   </joint>
   <!-- Gazebo Camera Plugin -->
   <gazebo reference="camera_link">
+    <!-- <plugin filename="gz_ros2_control-system" name="gz_ros_2_control::GazeboSimROS2ControlPlugin">
+      <robot_param_node>robot_state_publisher</robot_param_node>
+      <parameters>$(find tool_tracker)/config/panda_controllers.yaml</parameters>
+    </plugin> -->
+    <!-- <plugin filename="gz_ros2_control-system" name="gz_ros_2_control::GazeboSimROS2ControlPlugin">
+      <robot_param_node>robot_state_publisher</robot_param_node>
+      <parameters>$(arg ros_control_config)</parameters>
+    </plugin> -->
     <sensor type="camera" name="overhead_camera">
       <always_on>true</always_on>

Commit message: Resolved the issue of consuming image frame and live displaying it in gazebo

File: src/tool_tracker/urdf/simulation_scene.xacro (robot description, xacro)
@@ -1,13 +1,16 @@
 <?xml version="1.0" encoding="UTF-8"?>
-<robot name="panda_vision_stage" xmlns:xacro="http://www.ros.org/wiki/xacro">
-  <!-- 1. Include Pre-installed Panda Xacro -->
+<robot name="panda_tracker" xmlns:xacro="http://www.w3.org/2001/XMLSchema-instance">
   <xacro:include filename="$(find tool_tracker)/urdf/panda.urdf" />
-  <!-- <xacro:include filename="$(find moveit_resources_panda_description)/urdf/panda.urdf" />
-  <xacro:include filename="$(find moveit_resources_panda_description)/urdf/panda_ros2_control.xacro" /> -->
-  <!-- <xacro:panda_ros2_control
-    name="PandaGazeboHardware"
-    plugin_name="gz_ros2_control/GazeboSimSystem" /> -->
-  <!-- 2. Single Root Link Definition -->
-  <link name="world"/>
+  <material name="red">
+    <color rgba="1 0 0 1"/>
+  </material>
+  <gazebo>
+    <plugin
+      filename="ignition-gazebo-sensors-system"
+      name="ignition::gazebo::systems::Sensors">
+      <render_engine>ogre2</render_engine>
+    </plugin>
+  </gazebo>
+  <link name="world"></link>
   <joint name="world_to_panda" type="fixed">
     <parent link="world"/>
@@ -15,50 +18,54 @@
     <origin xyz="0 0 0" rpy="0 0 0"/>
   </joint>
-  <!-- 3. Fixed Overhead Camera Looking at End-Effector -->
   <link name="camera_link">
     <visual>
-      <geometry><box size="0.05 0.05 0.05"/></geometry>
+      <geometry>
+        <box size="0.015 0.08 0.08"/>
+      </geometry>
+      <material name="red" />
     </visual>
     <collision>
       <geometry>
-        <box size="0.05 0.05 0.05"/>
+        <box size="0.015 0.08 0.08"/>
       </geometry>
     </collision>
     <inertial>
       <origin xyz="0 0 0" rpy="0 0 0"/>
-      <mass value="1.0"/>
-      <inertia ixx="0.01" iyy="0.01" izz="0.01" ixy="0" ixz="0" iyz="0"/>
+      <mass value="2"/>
+      <inertia ixx="0.01" ixy="0" ixz="0" iyy="0.01" iyz="0" izz="0.01"/>
     </inertial>
   </link>
-  <joint name="world_to_camera" type="fixed">
+  <joint name="camera_joint" type="fixed">
     <parent link="world"/>
     <child link="camera_link"/>
-    <origin xyz="0.8 0.0 1.2" rpy="0 0.785 3.14159"/>
+    <origin xyz="0.900 0 0.995" rpy="0 -0.4 0"/>
   </joint>
-  <!-- Gazebo Camera Plugin -->
+  <link name="camera_link_optical"></link>
+  <joint name="camera_optical_joint" type="fixed">
+    <parent link="camera_link"/>
+    <child link="camera_link_optical"/>
+    <!-- Standard ROS to Optical Frame Transform: -90 deg roll, -90 deg yaw -->
+    <origin xyz="0 0 0" rpy="-1.57079632679 0 -1.57079632679"/>
+  </joint>
   <gazebo reference="camera_link">
-    <!-- <plugin filename="gz_ros2_control-system" name="gz_ros_2_control::GazeboSimROS2ControlPlugin">
-      <robot_param_node>robot_state_publisher</robot_param_node>
-      <parameters>$(find tool_tracker)/config/panda_controllers.yaml</parameters>
-    </plugin> -->
-    <!-- <plugin filename="gz_ros2_control-system" name="gz_ros_2_control::GazeboSimROS2ControlPlugin">
-      <robot_param_node>robot_state_publisher</robot_param_node>
-      <parameters>$(arg ros_control_config)</parameters>
-    </plugin> -->
-    <sensor type="camera" name="overhead_camera">
+    <sensor name="camera" type="camera">
+      <pose>0 0 0 0 0 0</pose>
+      <visualize>true</visualize>
       <always_on>true</always_on>
-      <update_rate>30.0</update_rate>
+      <update_rate>10</update_rate>
       <topic>camera/image_raw</topic>
       <camera>
-        <horizontal_fov>1.047</horizontal_fov>
+        <camera_info_topic>camera/camera_info</camera_info_topic>
+        <horizontal_fov>1.089</horizontal_fov>
         <image>
+          <format>R8G8B8</format>
           <width>640</width>
           <height>480</height>
-          <format>R8G8B8</format>
         </image>
         <clip>
-          <far>0.1</far>
-          <near>100.0</near>
+          <near>0.05</near>
+          <far>8.0</far>
         </clip>
+        <gz_frame_id>camera_link_optical</gz_frame_id>
       </camera>
     </sensor>

Commit message: Corrected the camera's position

File: src/tool_tracker/urdf/simulation_scene.xacro (robot description, xacro)
@@ -39,5 +39,5 @@
     <parent link="world"/>
     <child link="camera_link"/>
-    <origin xyz="0.900 0 0.995" rpy="0 -0.4 0"/>
+    <origin xyz="0.8 0.0 1.2" rpy="0 0.785 3.14159"/>
   </joint>
   <link name="camera_link_optical"></link>

Commit message: implemented a looping motion for the robot

File: src/tool_tracker/urdf/simulation_scene.xacro (robot description, xacro)
@@ -1,5 +1,27 @@
 <?xml version="1.0" encoding="UTF-8"?>
-<robot name="panda_tracker" xmlns:xacro="http://www.w3.org/2001/XMLSchema-instance">
+<robot name="panda_tracker" xmlns:xacro="http://www.ros.org/wiki/xacro">
   <xacro:include filename="$(find tool_tracker)/urdf/panda.urdf" />
+  <xacro:macro name="panda_joint_position_controller" params="joint_name effort_limit">
+    <gazebo>
+      <plugin
+        filename="ignition-gazebo-joint-position-controller-system"
+        name="ignition::gazebo::systems::JointPositionController">
+        <joint_name>${joint_name}</joint_name>
+        <topic>/model/panda_tracker/joint/${joint_name}/cmd_pos</topic>
+        <p_gain>100</p_gain>
+        <i_gain>0</i_gain>
+        <d_gain>10</d_gain>
+        <cmd_max>${effort_limit}</cmd_max>
+        <cmd_min>-${effort_limit}</cmd_min>
+      </plugin>
+    </gazebo>
+  </xacro:macro>
+  <xacro:panda_joint_position_controller joint_name="panda_joint1" effort_limit="87" />
+  <xacro:panda_joint_position_controller joint_name="panda_joint2" effort_limit="87" />
+  <xacro:panda_joint_position_controller joint_name="panda_joint3" effort_limit="87" />
+  <xacro:panda_joint_position_controller joint_name="panda_joint4" effort_limit="87" />
+  <xacro:panda_joint_position_controller joint_name="panda_joint5" effort_limit="12" />
+  <xacro:panda_joint_position_controller joint_name="panda_joint6" effort_limit="12" />
+  <xacro:panda_joint_position_controller joint_name="panda_joint7" effort_limit="12" />
   <material name="red">
     <color rgba="1 0 0 1"/>

Commit message: Adjusted camera's position to have the view of end-effector

File: src/tool_tracker/urdf/simulation_scene.xacro (robot description, xacro)
@@ -61,5 +61,5 @@
     <parent link="world"/>
     <child link="camera_link"/>
-    <origin xyz="0.8 0.0 1.2" rpy="0 0.785 3.14159"/>
+    <origin xyz="1.15 -1.5 1.3" rpy="0 0.356 2.111"/>
   </joint>
   <link name="camera_link_optical"></link>
@@ -79,5 +79,5 @@
       <camera>
         <camera_info_topic>camera/camera_info</camera_info_topic>
-        <horizontal_fov>1.089</horizontal_fov>
+        <horizontal_fov>1.3</horizontal_fov>
         <image>
           <format>R8G8B8</format>

Commit message: improved frame update rate, changed trajectory to drawing a circle

File: src/tool_tracker/urdf/simulation_scene.xacro (robot description, xacro)
@@ -61,6 +61,6 @@
     <parent link="world"/>
     <child link="camera_link"/>
-    <!-- In front of the raised marker path, centered and aimed slightly down. -->
-    <origin xyz="1.35 -0.12 0.37" rpy="0 0 3.14159265359"/>
+    <!-- Aim at the elevated circle, which lies in the camera image plane (world Y-Z). -->
+    <origin xyz="1.42 -0.12 0.33" rpy="0 0 3.14159265359"/>
   </joint>
   <link name="camera_link_optical"></link>
@@ -75,5 +75,5 @@
       <visualize>true</visualize>
       <always_on>true</always_on>
-      <update_rate>10</update_rate>
+      <update_rate>30</update_rate>
       <topic>camera/image_raw</topic>
       <camera>

Commit message: modifed the trajectory and cam's position

File: src/tool_tracker/urdf/simulation_scene.xacro (robot description, xacro)
@@ -61,6 +61,6 @@
     <parent link="world"/>
     <child link="camera_link"/>
-    <!-- Aim at the elevated circle, which lies in the camera image plane (world Y-Z). -->
-    <origin xyz="1.42 -0.12 0.33" rpy="0 0 3.14159265359"/>
+    <!-- Aim at the elevated, camera-facing circle in front of the robot. -->
+    <origin xyz="1.42 0 0.33" rpy="0 0 3.111"/>
   </joint>
   <link name="camera_link_optical"></link>
